Commit message: new project structure & added teachbot

File: my_uf_moveit_config/config/lite6_robot.ros2_control.xacro (robot description, xacro)
@@ -1,10 +1,16 @@
 <?xml version="1.0"?>
 <robot xmlns:xacro="http://www.ros.org/wiki/xacro">
-    <xacro:macro name="lite6_robot_ros2_control" params="name initial_positions_file">
+    <xacro:macro name="lite6_robot_ros2_control" params="name initial_positions_file sim_gazebo:=false">
         <xacro:property name="initial_positions" value="${load_yaml(initial_positions_file)['initial_positions']}"/>
         <ros2_control name="${name}" type="system">
             <hardware>
-                <!-- By default, set up controllers for simulation. This won't work on real hardware -->
-                <plugin>mock_components/GenericSystem</plugin>
+                <xacro:if value="${sim_gazebo}">
+                    <!-- Gazebo simulation -->
+                    <plugin>gz_ros2_control/GazeboSimSystem</plugin>
+                </xacro:if>
+                <xacro:unless value="${sim_gazebo}">
+                    <!-- Fake/mock hardware for testing -->
+                    <plugin>mock_components/GenericSystem</plugin>
+                </xacro:unless>
             </hardware>
             <joint name="joint1">

File: my_uf_moveit_config/config/lite6_robot.urdf.xacro (robot description, xacro)
@@ -2,8 +2,9 @@
 <robot xmlns:xacro="http://www.ros.org/wiki/xacro" name="lite6_robot">
     <xacro:arg name="initial_positions_file" default="initial_positions.yaml" />
+    <xacro:arg name="sim_gazebo" default="false" />
     <!-- Import lite6_robot urdf file -->
     <xacro:include filename="$(find my_uf_description)/urdf/lite6_robot.urdf.xacro" />
     <!-- Import control_xacro -->
     <xacro:include filename="lite6_robot.ros2_control.xacro" />
-    <xacro:lite6_robot_ros2_control name="FakeSystem" initial_positions_file="$(arg initial_positions_file)"/>
+    <xacro:lite6_robot_ros2_control name="FakeSystem" initial_positions_file="$(arg initial_positions_file)" sim_gazebo="$(arg sim_gazebo)"/>
 </robot>

Commit message: 20260105

File: my_uf_moveit_config/config/lite6_robot.ros2_control.xacro (robot description, xacro)
@@ -1,16 +1,10 @@
 <?xml version="1.0"?>
 <robot xmlns:xacro="http://www.ros.org/wiki/xacro">
-    <xacro:macro name="lite6_robot_ros2_control" params="name initial_positions_file sim_gazebo:=false">
-        <xacro:property name="initial_positions" value="${load_yaml(initial_positions_file)['initial_positions']}"/>
+    <xacro:macro name="lite6_robot_ros2_control" params="name initial_positions_file">
+        <xacro:property name="initial_positions" value="${xacro.load_yaml(initial_positions_file)['initial_positions']}"/>
         <ros2_control name="${name}" type="system">
             <hardware>
-                <xacro:if value="${sim_gazebo}">
-                    <!-- Gazebo simulation -->
-                    <plugin>gz_ros2_control/GazeboSimSystem</plugin>
-                </xacro:if>
-                <xacro:unless value="${sim_gazebo}">
-                    <!-- Fake/mock hardware for testing -->
-                    <plugin>mock_components/GenericSystem</plugin>
-                </xacro:unless>
+                <!-- By default, set up controllers for simulation. This won't work on real hardware -->
+                <plugin>mock_components/GenericSystem</plugin>
             </hardware>
             <joint name="joint1">

File: my_uf_moveit_config/config/lite6_robot.urdf.xacro (robot description, xacro)
@@ -3,5 +3,7 @@
     <xacro:arg name="initial_positions_file" default="initial_positions.yaml" />
     <!-- Import lite6_robot urdf file -->
-    <!-- This already includes ros2_control from xarm_description -->
     <xacro:include filename="$(find my_uf_description)/urdf/lite6_robot.urdf.xacro" />
+    <!-- Import control_xacro -->
+    <xacro:include filename="lite6_robot.ros2_control.xacro" />
+    <xacro:lite6_robot_ros2_control name="FakeSystem" initial_positions_file="$(arg initial_positions_file)"/>
 </robot>
