Commit message: Added branch jazzy-xarm5

File: my_uf_description/urdf/uf_robot.urdf.xacro (robot description, xacro)
@@ -1,4 +1,4 @@
 <?xml version="1.0"?>
-<robot xmlns:xacro="http://wiki.ros.org/xacro" name="lite6_robot">
+<robot xmlns:xacro="http://wiki.ros.org/xacro" name="uf_robot">
   <xacro:arg name="prefix" default=""/>
   <xacro:arg name="hw_ns" default=""/>
@@ -6,10 +6,10 @@
   <xacro:arg name="effort_control" default="false"/>
   <xacro:arg name="velocity_control" default="false"/>
-  <xacro:arg name="add_gripper" default="false"/>
-  <xacro:arg name="add_vacuum_gripper" default="true"/>
+  <xacro:arg name="add_gripper" default="true"/>
+  <xacro:arg name="add_vacuum_gripper" default="false"/>
   <xacro:arg name="model1300" default="false"/>
   <xacro:arg name="dof" default="6"/>
   <xacro:arg name="robot_ip" default=""/>
-  <xacro:arg name="robot_type" default="lite"/>
+  <xacro:arg name="robot_type" default="xarm"/>
   <xacro:arg name="robot_sn" default=""/>
   <xacro:arg name="report_type" default="normal"/>
@@ -46,4 +46,6 @@
                      effort_control="$(arg effort_control)"
                      velocity_control="$(arg velocity_control)"
+                     add_gripper="$(arg add_gripper)"
+                     add_vacuum_gripper="$(arg add_vacuum_gripper)"
                      dof="$(arg dof)"
                      ros2_control_plugin="$(arg ros2_control_plugin)"

File: my_uf_moveit_config/config/backup/lite6_robot.urdf.xacro (robot description, xacro)
@@ -1,9 +1,9 @@
 <?xml version="1.0"?>
-<robot xmlns:xacro="http://www.ros.org/wiki/xacro" name="lite6_robot">
+<robot xmlns:xacro="http://www.ros.org/wiki/xacro" name="uf_robot">
     <xacro:arg name="initial_positions_file" default="initial_positions.yaml" />
-    <!-- Import lite6_robot urdf file -->
-    <xacro:include filename="$(find my_uf_description)/urdf/lite6_robot.urdf.xacro" />
+    <!-- Import uf_robot urdf file -->
+    <xacro:include filename="$(find my_uf_description)/urdf/uf_robot.urdf.xacro" />
     <!-- Import control_xacro -->
-    <xacro:include filename="lite6_robot.ros2_control.xacro" />
-    <xacro:lite6_robot_ros2_control name="FakeSystem" initial_positions_file="$(arg initial_positions_file)"/>
+    <xacro:include filename="uf_robot.ros2_control.xacro" />
+    <xacro:uf_robot_ros2_control name="FakeSystem" initial_positions_file="$(arg initial_positions_file)"/>
 </robot>

File: my_uf_moveit_config/config/uf_robot.ros2_control.xacro (robot description, xacro)
@@ -1,5 +1,5 @@
 <?xml version="1.0"?>
 <robot xmlns:xacro="http://www.ros.org/wiki/xacro">
-    <xacro:macro name="lite6_robot_ros2_control" params="name initial_positions_file">
+    <xacro:macro name="uf_robot_ros2_control" params="name initial_positions_file">
         <xacro:property name="initial_positions" value="${xacro.load_yaml(initial_positions_file)['initial_positions']}"/>
         <ros2_control name="${name}" type="system">

Commit message: Added branch jazzy-xarm5

File: my_uf_description/urdf/uf_robot.urdf.xacro (robot description, xacro)
@@ -115,4 +115,5 @@
       <xacro:box_inertia m="20" x="0.7" y="1.1" z="0.03"/>
     </inertial>
+    <!--
     <collision>
       <origin xyz="0 0 0.0" />
@@ -121,8 +122,10 @@
       </geometry>
     </collision>
+    -->
   </link>
   <!-- dit is niet juist parent en child zijn omgedraaid -->
   <joint name="baseplate_joint" type="fixed">
-    <origin xyz="0 0 0.015" />
+    <!--<origin xyz="0 0 0.015" /> -->
+      <origin xyz="0 0 -1.0" />
     <parent link="world" />
     <child link="baseplate_link" />
@@ -148,5 +151,5 @@
   <joint name="mountingplate_joint" type="fixed">
     <origin xyz="-0.285 0.0 0.0175" />
-    <parent link="baseplate_link" />
+    <parent link="world" />
     <child link="mountingplate_link" />
   </joint>
@@ -154,5 +157,6 @@
   </link >
   <joint name="base_plate_to_xarm_joint" type="fixed">
-    <origin xyz="-0.0 0.0 0.0025" />
+    <!--<origin xyz="-0.0 0.0 0.0025" />-->
+    <origin xyz="-0.0 0.0 0.5" />
     <parent link="mountingplate_link" />
     <child link="xarm_link" />

File: my_uf_moveit_config/config/uf_robot.urdf.xacro (robot description, xacro)
@@ -1,5 +1,9 @@
 <?xml version="1.0"?>
 <robot xmlns:xacro="http://www.ros.org/wiki/xacro" name="uf_robot">
+    <xacro:arg name="initial_positions_file" default="initial_positions.yaml" />
     <!-- Import uf_robot urdf file -->
     <xacro:include filename="$(find my_uf_description)/urdf/uf_robot.urdf.xacro" />
+    <!-- Import control_xacro -->
+    <xacro:include filename="uf_robot.ros2_control.xacro" />
+    <xacro:uf_robot_ros2_control name="FakeSystem" initial_positions_file="$(arg initial_positions_file)"/>
 </robot>

Commit message: 20260318

File: my_uf_description/urdf/uf_robot.urdf.xacro (robot description, xacro)
@@ -9,5 +9,5 @@
   <xacro:arg name="add_vacuum_gripper" default="false"/>
   <xacro:arg name="model1300" default="false"/>
-  <xacro:arg name="dof" default="6"/>
+  <xacro:arg name="dof" default="5"/>
   <xacro:arg name="robot_ip" default=""/>
   <xacro:arg name="robot_type" default="xarm"/>
@@ -115,5 +115,4 @@
       <xacro:box_inertia m="20" x="0.7" y="1.1" z="0.03"/>
     </inertial>
-    <!--
     <collision>
       <origin xyz="0 0 0.0" />
@@ -122,10 +121,8 @@
       </geometry>
     </collision>
-    -->
   </link>
   <!-- dit is niet juist parent en child zijn omgedraaid -->
   <joint name="baseplate_joint" type="fixed">
-    <!--<origin xyz="0 0 0.015" /> -->
-      <origin xyz="0 0 -1.0" />
+    <origin xyz="0 0 0.015" />
     <parent link="world" />
     <child link="baseplate_link" />
@@ -135,5 +132,5 @@
       <origin xyz="0 0 0.0" />
       <geometry>
-        <box size="0.130 0.190 0.005" />
+        <box size="0.130 0.190 0.100" />
       </geometry>
       <material name="red"/>
@@ -150,6 +147,6 @@
   </link>
   <joint name="mountingplate_joint" type="fixed">
-    <origin xyz="-0.285 0.0 0.0175" />
-    <parent link="world" />
+    <origin xyz="-0.285 0.0 0.065" />
+    <parent link="baseplate_link" />
     <child link="mountingplate_link" />
   </joint>
@@ -157,6 +154,5 @@
   </link >
   <joint name="base_plate_to_xarm_joint" type="fixed">
-    <!--<origin xyz="-0.0 0.0 0.0025" />-->
-    <origin xyz="-0.0 0.0 0.5" />
+    <origin xyz="-0.0 0.0 0.05" />
     <parent link="mountingplate_link" />
     <child link="xarm_link" />

File: my_uf_moveit_config/config/uf_robot.ros2_control.xacro (robot description, xacro)
@@ -43,11 +43,4 @@
                 <state_interface name="velocity"/>
             </joint>
-            <joint name="joint6">
-                <command_interface name="position"/>
-                <state_interface name="position">
-                  <param name="initial_value">${initial_positions['joint6']}</param>
-                </state_interface>
-                <state_interface name="velocity"/>
-            </joint>
         </ros2_control>
     </xacro:macro>

File: my_uf_moveit_config/config/uf_robot.urdf.xacro (robot description, xacro)
@@ -1,9 +1,5 @@
 <?xml version="1.0"?>
 <robot xmlns:xacro="http://www.ros.org/wiki/xacro" name="uf_robot">
-    <xacro:arg name="initial_positions_file" default="initial_positions.yaml" />
     <!-- Import uf_robot urdf file -->
     <xacro:include filename="$(find my_uf_description)/urdf/uf_robot.urdf.xacro" />
-    <!-- Import control_xacro -->
-    <xacro:include filename="uf_robot.ros2_control.xacro" />
-    <xacro:uf_robot_ros2_control name="FakeSystem" initial_positions_file="$(arg initial_positions_file)"/>
 </robot>
